File: Artwork/Artwork-CAD/BHVBadge.kicad_pcb (KiCad board)
At the start: 2 copper layers, 116.2 x 144.6 mm, 8 parts

Commit message: Artwork
Parts:
- removed the G*** at (0.00, 0.00) (x7)
- added G*** (x7): LOGO, LOGO, F.Cu at (0.00, 0.00)
- moved ? 1272.0 mm to (-1619.6, -595.0)
Other:
- board size 116.2 x 144.6 mm -> 101.1 x 125.8 mm
