File: Artwork/Artwork-CAD/BHVBadge.kicad_pcb (KiCad board)
At the start: 2 copper layers, 101.1 x 125.8 mm, 8 parts

Commit message: Finalizing Proto
Parts:
- removed the G*** at (0.00, 0.00) (x7)
- added G*** (x7): LOGO, LOGO, F.Cu at (98.9, 67.9)
- added REF**: 3.5mm, BadgePirates:Hole_3.5mm, F.Cu at (118.2, 23.4)
- moved ? 101.1 mm to (-1518.5, -595.0)
Other:
- outline, holes or cut-outs redrawn
- net class Default removed
