File: CAD/BiohackingPivot.kicad_pcb (KiCad board)
At the start: 2 copper layers, 10 parts, among them SW1 SW_DP3T

Commit message: Finalizing Proto
Parts:
- removed SW1: SW_DP3T, Button_Switch_SMD:SW_SP3T_PCM13
- added D10: LED, BadgePirates:LED_D5.0mm, B.Cu at (95.2, 98.0)
- added D11: LED, BadgePirates:LED_D5.0mm, B.Cu at (116.2, 55.4)
- added D12: LED, BadgePirates:LED_D5.0mm, B.Cu at (140.9, 53.9)
- added D13: LED, BadgePirates:LED_D5.0mm, B.Cu at (153.4, 56.3)
- added D7: LED, BadgePirates:LED_D5.0mm, B.Cu at (104.7, 62.4)
- added D8: LED, BadgePirates:LED_D5.0mm, B.Cu at (97.3, 72.7)
- added D9: LED, BadgePirates:LED_D5.0mm, B.Cu at (94.0, 85.4)
- added G*** (x7): LOGO, LOGO, F.Cu at (109.4, 92.9)
- added G***: fg, BadgePiratesLogos:FG_B.Cu, F.Cu at (169.3, 135.6)
- added G***: NG_BSilk_B.Cu, BadgePiratesLogos:NG_B.Cu, F.Cu at (151.4, 143.1)
- added G***: BP Logo, BadgePiratesLogos:BPSkull_Distressed_B.SILK, F.Cu at (112.7, 116.0)
- added G***: LOGO, BadgePiratesLogos:BadgePiratesURL_B.SLK, F.Cu at (112.7, 109.1)
- added REF**: 3.5mm, BadgePirates:Hole_3.5mm, F.Cu at (128.7, 48.5)
- added RN3: 1k_Array, Resistor_SMD:R_Array_Convex_4x1206, B.Cu at (127.3, 108.3)
- added RN4: 1k_Array, Resistor_SMD:R_Array_Convex_4x1206, B.Cu at (136.1, 64.6)
- added SW3: SW-SP4T, BadgePirates:SP4T - CUS-14TB, B.Cu at (113.6, 133.0)
- BT1: footprint BadgePirates:BatteryHolder_MPD_BC2003_1x2032_Fixed -> BadgePirates:BATHLD006SMT - CR2450
- moved BT1 40.8 mm to (138.2, 125.6)
- moved D3 39.3 mm to (169.8, 107.0), turned to 180 degrees
- moved D1 36.3 mm to (152.3, 98.2), turned to 180 degrees
- moved RN2 31.2 mm to (161.6, 78.1), turned to -90 degrees
- moved RN1 30.2 mm to (162.9, 119.8), turned to 90 degrees
- moved D5 28.4 mm to (157.8, 89.1), turned to 180 degrees
- moved D4 22.3 mm to (158.4, 106.5), turned to 180 degrees
- moved D2 21.2 mm to (170.1, 90.8), turned to 180 degrees
- moved D6 8.69 mm to (172.8, 98.8), turned to 180 degrees
Connections:
- net Net-(RN1-R1.1) renamed WHITE
- net Net-(RN2-R1.1) renamed UV
Routing:
- net BLINKIE: track 0.00 -> 132.8 mm
- net UV: track 0.00 -> 116.8 mm
- net Net-(D7-A): track 0.00 -> 72.9 mm
- net Net-(D8-A): track 0.00 -> 63.6 mm
- net +3.3V: track 0.00 -> 63.3 mm
- net WHITE: track 0.00 -> 61.8 mm
- net Net-(D9-A): track 0.00 -> 54.4 mm
- net Net-(D10-A): track 0.00 -> 37.3 mm
- net Net-(D3-A): track 0.00 -> 34.9 mm
- net Net-(D5-A): track 0.00 -> 32.2 mm
- net Net-(D1-A): track 0.00 -> 26.8 mm
- net Net-(D6-A): track 0.00 -> 22.9 mm
- net Net-(D11-A): track 0.00 -> 22.7 mm
- net Net-(D13-A): track 0.00 -> 21.9 mm
- net Net-(D2-A): track 0.00 -> 15.2 mm
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- added copper zone on B.Cu, net GND
Other:
- board outline added: 101.1 x 125.8 mm
- rule pad_to_mask_clearance: 0 -> 0.2
