File: CAD/BiohackingPivot.kicad_pcb (KiCad board)
At the start: 2 copper layers, 101.1 x 125.8 mm, 47 parts, among them SW3 SW-SP4T

Commit message: fixes
Parts:
- D4, D5, D6: value LED -> WHITE
- REF**: value 3.5mm -> 4mm
- RN1, RN2, RN3, RN4: footprint Resistor_SMD:R_Array_Convex_4x1206 -> Resistor_SMD:R_Array_Convex_4x0603
- moved G*** 5.04 mm to (156.7, 108.7), turned to -45 degrees
- moved G*** 4.87 mm to (171.7, 109.1), turned to 40 degrees
- moved G*** 4.14 mm to (154.0, 88.3), turned to -140 degrees
- moved G*** 3.99 mm to (149.2, 98.4), turned to -90 degrees
- moved G*** 3.94 mm to (175.2, 99.2), turned to 90 degrees
- moved REF** 2.40 mm to (128.6, 50.9)
- moved D5 2.12 mm to (156.3, 90.5), turned to -140 degrees
- moved G*** 1.19 mm to (171.1, 89.1), turned to 135 degrees
- moved RN2 1.08 mm to (160.8, 77.5)
- moved RN3 0.92 mm to (127.7, 109.2), turned to 90 degrees
- moved RN1 0.85 mm to (163.8, 119.5)
- moved RN4 0.76 mm to (135.5, 64.1)
- turned D1 to -90 degrees
- turned D2 to 135 degrees
- turned D3 to 40 degrees
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Connections:
- D10 pad 1: unconnected-(D10-K-Pad1) -> GND
- D11 pad 1: unconnected-(D11-K-Pad1) -> GND
- D12 pad 1: unconnected-(D12-K-Pad1) -> GND
- D13 pad 1: unconnected-(D13-K-Pad1) -> GND
- D7 pad 1: unconnected-(D7-K-Pad1) -> GND
- D8 pad 1: unconnected-(D8-K-Pad1) -> GND
- D9 pad 1: unconnected-(D9-K-Pad1) -> GND
Routing:
- net UV: track 116.8 -> 122.8 mm
- net Net-(D3-A): track 34.9 -> 40.1 mm
- net Net-(D10-A): track 37.3 -> 41.9 mm
- net BLINKIE: track 132.8 -> 128.4 mm
- net GND: track 2.94 -> 6.18 mm, vias 2 -> 4
- net Net-(D2-A): track 15.2 -> 18.2 mm
- net Net-(D6-A): track 22.9 -> 24.9 mm
- net WHITE: track 61.8 -> 63.6 mm
- net Net-(D1-A): track 26.8 -> 28.3 mm
- net Net-(D5-A): track 32.2 -> 30.8 mm
- net Net-(D9-A): track 54.4 -> 55.8 mm
- net Net-(D7-A): track 72.9 -> 71.7 mm, vias 0 -> 2
- net Net-(D13-A): track 21.9 -> 22.9 mm
- net Net-(D4-A): track 14.7 -> 15.3 mm
- net Net-(D8-A): track 63.6 -> 64.0 mm, vias 0 -> 2
Other:
- outline, holes or cut-outs redrawn
- board text added: "CR-2450"
- board text added: "Lee Cyborg"
- board text removed: "CR-2032"
- board text removed: "leeborg"
