File: CAD/altBiohackingPivot.kicad_pcb (KiCad board)
At the start: 2 copper layers, 101.1 x 125.8 mm, 47 parts, among them SW3 SW-SP4T

Commit message: alt layout
Parts:
- BT1: value Battery_Cell -> CR 2450
- D1, D2, D3: value UV -> UV LED; footprint LED_SMD:LED_0805_2012Metric -> LED_SMD:LED_1206_3216Metric
- D4, D5, D6: value LED -> White
- moved D2 0.45 mm to (170.1, 90.8)
- moved D3 0.41 mm to (169.8, 107.0)
- moved D1 0.22 mm to (152.3, 98.2)
- renumbered SW3 to Blinkie/Off/White/UV
Other:
- board text removed: "BLINKIE/OFF/WHITE/UV"
- board text removed: "CR-2032"
