File: CAD/BiohackingPivot.kicad_sch (KiCad schematic)
At the start: 10 parts, among them SW1 SW_DP3T

Commit message: Finalizing Proto
Parts:
- removed SW1: SW_DP3T, Button_Switch_SMD:SW_SP3T_PCM13, symbol Switch:SW_DP3T
- added D10, D11, D12, D13, D7, D8, D9: LED, BadgePirates:LED_D5.0mm, symbol BadgePiratesSymbolLibrary:LED
- added RN3, RN4: 1k_Array, Resistor_SMD:R_Array_Convex_4x1206, symbol BadgePiratesSymbolLibrary:R_Pack04
- added SW3: SW-SP4T, BadgePirates:SP4T - CUS-14TB, symbol BadgePiratesSymbolLibrary:SP4T
- BT1: footprint BadgePirates:BatteryHolder_MPD_BC2003_1x2032_Fixed -> BadgePirates:BATHLD006SMT - CR2450
Connections:
- net +3.3V: now also SW3.4
- net WHITE: now reaches RN1.1 (R1.1), RN1.2 (R2.1), RN1.3 (R3.1)
- net WHITE: now also SW3.2
- net UV: now reaches RN2.1 (R1.1), RN2.2 (R2.1), RN2.3 (R3.1)
- net UV: now also SW3.1
- new net: D7.2 (A), RN3.5 (R4.2)
- new net: D8.2 (A), RN3.6 (R3.2)
- new net: D9.2 (A), RN3.7 (R2.2)
- new net: D10.2 (A), RN3.8 (R1.2)
- new net: D11.2 (A), RN4.5 (R4.2)
- new net: D12.2 (A), RN4.6 (R3.2)
- new net: D13.2 (A), RN4.7 (R2.2)
- new net BLINKIE: RN3.1 (R1.1), RN3.2 (R2.1), RN3.3 (R3.1), RN3.4 (R4.1), RN4.2 (R2.1), RN4.3 (R3.1), RN4.4 (R4.1), SW3.5
- no-connect marks 5 -> 7
Other:
- note added: "Blinkie"
- note added: "UV"
- note removed: "IR"
- moved on the sheet: BT1, D4, D5, D6, RN1

Commit message: alt layout
Parts:
- D1, D2, D3: footprint LED_SMD:LED_1206_3216Metric -> LED_SMD:LED_0805_2012Metric

Commit message: fixes
Parts:
- RN1, RN2, RN3, RN4: footprint Resistor_SMD:R_Array_Convex_4x1206 -> Resistor_SMD:R_Array_Convex_4x0603
Connections:
- net GND: now also D10.1 (K), D11.1 (K), D12.1 (K), D13.1 (K), D7.1 (K), D8.1 (K), D9.1 (K)
Changed lines of the file:
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@@
 (kicad_sch (version 20230121) (generator eeschema)
   (paper "A4")
+  (junction (at 105.41 173.99) (diameter 0) (color 0 0 0 0)
+  )
   (junction (at 157.48 78.74) (diameter 0) (color 0 0 0 0)
   )
   (junction (at 161.29 149.86) (diameter 0) (color 0 0 0 0)
   )
+  (junction (at 105.41 182.88) (diameter 0) (color 0 0 0 0)
+  )
+  (junction (at 105.41 165.1) (diameter 0) (color 0 0 0 0)
+  )
   (junction (at 121.92 80.01) (diameter 0) (color 0 0 0 0)
   )
   (junction (at 161.29 144.78) (diameter 0) (color 0 0 0 0)
   )
+  (junction (at 105.41 156.21) (diameter 0) (color 0 0 0 0)
+  )
   (junction (at 161.29 158.75) (diameter 0) (color 0 0 0 0)
   )
   (junction (at 121.92 116.84) (diameter 0) (color 0 0 0 0)
+  )
+  (junction (at 105.41 148.59) (diameter 0) (color 0 0 0 0)
   )
   (junction (at 161.29 170.18) (diameter 0) (color 0 0 0 0)
@@
     (stroke (width 0) (type default))
   )
+  (wire (pts (xy 111.76 139.7) (xy 105.41 139.7))
+    (stroke (width 0) (type default))
+  )
+  (wire (pts (xy 105.41 139.7) (xy 105.41 148.59))
+    (stroke (width 0) (type default))
+  )
   (wire (pts (xy 146.05 170.18) (xy 161.29 170.18))
     (stroke (width 0) (type default))
@@
     (stroke (width 0) (type default))
   )
+  (wire (pts (xy 105.41 173.99) (xy 105.41 165.1))
+    (stroke (width 0) (type default))
+  )
   (wire (pts (xy 157.48 78.74) (xy 157.48 81.28))
     (stroke (width 0) (type default))
@@
     (stroke (width 0) (type default))
   )
+  (wire (pts (xy 113.03 173.99) (xy 105.41 173.99))
+    (stroke (width 0) (type default))
+  )
   (wire (pts (xy 161.29 142.24) (xy 161.29 144.78))
     (stroke (width 0) (type default))
@@
     (stroke (width 0) (type default))
   )
+  (wire (pts (xy 105.41 148.59) (xy 105.41 156.21))
+    (stroke (width 0) (type default))
+  )
   (wire (pts (xy 121.92 80.01) (xy 124.46 80.01))
     (stroke (width 0) (type default))
   )
+  (wire (pts (xy 105.41 165.1) (xy 111.76 165.1))
+    (stroke (width 0) (type default))
+  )
   (wire (pts (xy 134.62 80.01) (xy 132.08 80.01))
     (stroke (width 0) (type default))
@@
     (stroke (width 0) (type default))
   )
+  (wire (pts (xy 105.41 182.88) (xy 105.41 173.99))
+    (stroke (width 0) (type default))
+  )
   (wire (pts (xy 121.92 107.95) (xy 121.92 116.84))
     (stroke (width 0) (type default))
@@
     (stroke (width 0) (type default))
   )
+  (wire (pts (xy 111.76 156.21) (xy 105.41 156.21))
+    (stroke (width 0) (type default))
+  )
   (wire (pts (xy 123.19 182.88) (xy 120.65 182.88))
     (stroke (width 0) (type default))
@@
     (stroke (width 0) (type default))
   )
+  (wire (pts (xy 111.76 148.59) (xy 105.41 148.59))
+    (stroke (width 0) (type default))
+  )
   (wire (pts (xy 137.16 71.12) (xy 132.08 71.12))
     (stroke (width 0) (type default))
@@
     (stroke (width 0) (type default))
   )
+  (wire (pts (xy 113.03 193.04) (xy 105.41 193.04))
+    (stroke (width 0) (type default))
+  )
   (wire (pts (xy 161.29 158.75) (xy 163.83 158.75))
     (stroke (width 0) (type default))
@@
     (stroke (width 0) (type default))
   )
+  (wire (pts (xy 105.41 156.21) (xy 105.41 165.1))
+    (stroke (width 0) (type default))
+  )
   (wire (pts (xy 124.46 107.95) (xy 121.92 107.95))
     (stroke (width 0) (type default))
@@
     (stroke (width 0) (type default))
   )
+  (wire (pts (xy 113.03 182.88) (xy 105.41 182.88))
+    (stroke (width 0) (type default))
+  )
   (wire (pts (xy 157.48 119.38) (xy 149.86 119.38))
     (stroke (width 0) (type default))
@@
     (stroke (width 0) (type default))
   )
+  (wire (pts (xy 101.6 165.1) (xy 105.41 165.1))
+    (stroke (width 0) (type default))
+  )
   (wire (pts (xy 157.48 116.84) (xy 149.86 116.84))
     (stroke (width 0) (type default))
   )
+  (wire (pts (xy 105.41 193.04) (xy 105.41 182.88))
+    (stroke (width 0) (type default))
+  )
   (wire (pts (xy 132.08 125.73) (xy 139.7 125.73))
     (stroke (width 0) (type default))
@@
     (stroke (width 0) (type default))
   )
-  (rectangle (start 110.49 133.35) (end 154.94 196.85)
+  (rectangle (start 91.44 133.35) (end 175.26 196.85)
     (stroke (width 0) (type default))
     (fill (type none))
@@
       (effects (font (size 1.27 1.27)))
     )
-    (property "Footprint" "Resistor_SMD:R_Array_Convex_4x1206" (at 140.97 137.795 90)
+    (property "Footprint" "Resistor_SMD:R_Array_Convex_4x0603" (at 140.97 137.795 90)
       (effects (font (size 1.27 1.27)) hide)
     )
@@
     )
   )
+  (symbol (lib_id "power:GND") (at 101.6 165.1 270) (unit 1)
+    (in_bom yes) (on_board yes) (dnp no) (fields_autoplaced)
+    (property "Reference" "#PWR06" (at 95.25 165.1 0)
+      (effects (font (size 1.27 1.27)) hide)
+    )
+    (property "Value" "GND" (at 97.79 165.735 90)
+      (effects (font (size 1.27 1.27)) (justify right))
+    )
+    (property "Footprint" "" (at 101.6 165.1 0)
+      (effects (font (size 1.27 1.27)) hide)
+    )
+    (property "Datasheet" "" (at 101.6 165.1 0)
+      (effects (font (size 1.27 1.27)) hide)
+    )
+    (pin "1")
+    (instances
+      (project "BiohackingPivot"
+        (path "/233c7065-1d62-4414-ad68-540cbd677115"
+          (reference "#PWR06") (unit 1)
+        )
+      )
+    )
+  )
   (symbol (lib_id "power:+3.3V") (at 200.66 123.19 0) (unit 1)
     (in_bom yes) (on_board yes) (dnp no)
@@
       (effects (font (size 1.27 1.27)))
     )
-    (property "Footprint" "Resistor_SMD:R_Array_Convex_4x1206" (at 140.97 165.735 90)
+    (property "Footprint" "Resistor_SMD:R_Array_Convex_4x0603" (at 140.97 165.735 90)
       (effects (font (size 1.27 1.27)) hide)
     )
@@
       (effects (font (size 1.27 1.27)))
     )
-    (property "Footprint" "Resistor_SMD:R_Array_Convex_4x1206" (at 144.78 69.215 90)
+    (property "Footprint" "Resistor_SMD:R_Array_Convex_4x0603" (at 144.78 69.215 90)
       (effects (font (size 1.27 1.27)) hide)
     )
@@
       (effects (font (size 1.27 1.27)))
     )
-    (property "Footprint" "Resistor_SMD:R_Array_Convex_4x1206" (at 144.78 107.315 90)
-      (effects (font (size 1.27 1.27)) hide)
-    )
+    (property "Footprint" "Resistor_SMD:R_Array_Convex_4x0603" (at 144.78 107.315 90)
+      (effects (font (size 1.27 1.27)) hide)
+    )

Commit message: Cleaning up folder and page settings
Other:
- note added: "Battery"
- note added: "Switch"
- company: (none) -> Badge Pirates
- title: (none) -> BioHacking Badge
- moved on the sheet: BT1, D1, D10, D11, D12, D13, D2, D3, D4, D5, D6, D7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
